File: bosonator/boson/boson.kicad_sch (KiCad schematic)
At the start: 8 parts, among them P1 DF40HC(4.0)-80DS-0.4V(51), P2 USB_C_Plug_USB2.0, U1 AMS1117-3.3

Commit message: [Boson] Quick & dirty routing
Connections:
- net GND: now also C3.2, C4.2, U1.1 (GND)
Changed lines of the file:
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@@
     )
   )
-  (symbol (lib_id "power:GND") (at 76.2 101.6 0) (unit 1)
+  (symbol (lib_id "power:GND") (at 80.01 101.6 0) (unit 1)
     (in_bom yes) (on_board yes) (dnp no)
-    (property "Reference" "#PWR01" (at 76.2 107.95 0)
+    (property "Reference" "#PWR01" (at 80.01 107.95 0)
       (effects (font (size 1.27 1.27)) hide)
     )
-    (property "Value" "GND" (at 76.2 109.22 90)
+    (property "Value" "GND" (at 80.01 109.22 90)
       (effects (font (size 1.27 1.27)) (justify left))
     )
-    (property "Footprint" "" (at 76.2 101.6 0)
+    (property "Footprint" "" (at 80.01 101.6 0)
       (effects (font (size 1.27 1.27)) hide)
     )
-    (property "Datasheet" "" (at 76.2 101.6 0)
+    (property "Datasheet" "" (at 80.01 101.6 0)
       (effects (font (size 1.27 1.27)) hide)
     )
