File: bosonator/boson.kicad_pcb (KiCad board)
At the start: 2 copper layers, 21 x 21 mm, 8 parts, among them P1 DF40HC(4.0)-80DS-0.4V(51), P2 USB_C_Plug_USB2.0, U1 AMS1117-3.3

Commit message: [Boson] Misc. WIP bad.
Routing:
- net +3.3V: track 36.9 -> 0.00 mm, vias 2 -> 0
- net GND: track 38.4 -> 3.53 mm, vias 13 -> 12
- net Net-(U1-VI): track 16.7 -> 0.00 mm
- net /USB_D_P: track 14.4 -> 0.00 mm, vias 1 -> 0
- net /USB_D_N: track 12.5 -> 0.00 mm, vias 3 -> 0
- net Net-(P2-CC2): track 10.1 -> 0.00 mm, vias 2 -> 0
- net Net-(P2-CC1): track 6.56 -> 0.00 mm
Other:
- board text added: "Re-center connector"
